File: esp32_prototype_board/esp32_prototype_board.kicad_sch (KiCad schematic)
At the start: 70 parts, among them J1 USB-C USB2 sink, J2 EXT 5V IN, J4 microSD SPI, J6 SPI EXP, J7 I2C EXP, J8 GPIO EXP, Q1 SS8050/MMBT3904, Q2 SS8050/MMBT3904, Q3 MMBT3904, SW1 EN/RST, SW2 BOOT, U1 CH340C, U2 AP2112K-3.3, U3 ESP32-WROOM-32E, U4 MAX98357A blue module

Commit message: adding final PCB files
Parts:
- added C14: 100nF, Capacitor_SMD:C_0805_2012Metric, symbol SweetYaar:C
- added H1, H2, H3, H4: M3 mounting hole, MountingHole:MountingHole_3.2mm_M3, symbol Mechanical:MountingHole
- JP1: value 5V source select -> 5V source switch; footprint Connector_PinHeader_2.54mm:PinHeader_1x03_P2.54mm_Vertical -> SweetYaar:SW-SMD_MS-22D28-G020; symbol SweetYaar:CONN_01X03 -> SweetYaar:SW_DPDT_MS22D28_SINGLE
- JP2: renamed from SJ1; value GPIO2 LED EN -> GPIO2 LED SW; footprint Jumper:SolderJumper-2_P1.3mm_Open_TrianglePad1.0x1.5mm -> SweetYaar:SW-SMD_MS-22D28-G020; symbol SweetYaar:JUMPER_2 -> SweetYaar:SW_DPDT_MS22D28_SINGLE
Connections:
- net 5V_SYS: now also C14.1
- net GND: now also C14.2
- no-connect marks 18 -> 19
