File: hardware/debugger/SweetYaarDebugger.kicad_pcb (KiCad board)
At the start: 2 copper layers, 50.1 x 18.6 mm, 19 parts, among them U1 USBLC6-2SC6

Commit message: Flipping debugger output connector
Parts:
- moved J_PROG1 12.7 mm to (113.3, 52.2), turned to 180 degrees
- moved JP2 10.1 mm to (105.2, 42.3)
- moved R1 8.09 mm to (100.0, 50.9), turned to 0 degrees
- moved JP1 2.31 mm to (105.3, 45.8)
Routing:
- net /BOOT: track 8.04 -> 10.5 mm, vias 0 -> 2
- net /UART_RXD: track 28.1 -> 29.4 mm
- net /3V3_REF: track 13.9 -> 13.0 mm
- net /UART_TXD: track 26.9 -> 27.7 mm
- net GND: track 29.6 -> 28.9 mm
- net Net-(D1-A): track 5.19 -> 5.61 mm, vias 2 -> 0
- net /ESP_EN: track 9.66 -> 9.29 mm, vias 2 -> 0

Commit message: Fixing rotation and position offsets
Parts:
- J_USB1: footprint Connector_USB:USB_C_Receptacle_HRO_TYPE-C-31-M-12 -> SweetYaar:USB_C_Receptacle_HRO_TYPE-C-31-M-12 - C165948
- U1: footprint Package_TO_SOT_SMD:SOT-23-6 -> SweetYaar:SOT-23-6 - USBLC6-2SC6 - C7519

Commit message: Creating production v1.0 manufacturing files
Parts:
- C2, C4: value 2.2uF -> 4.7uF
Changed lines of the file:
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@@
 		(sheetname "/")
 		(sheetfile "SweetYaarDebugger.kicad_sch")
+		(units
+			(unit
+				(name "A")
+				(pins "1" "2" "3" "4" "5" "6")
+			)
+		)
 		(attr through_hole dnp)
 		(duplicate_pad_numbers_are_jumpers no)
@@
 		(sheetname "/")
 		(sheetfile "SweetYaarDebugger.kicad_sch")
+		(units
+			(unit
+				(name "A")
+				(pins "1" "3" "2")
+			)
+		)
 		(attr smd)
 		(duplicate_pad_numbers_are_jumpers no)
@@
 		(sheetname "/")
 		(sheetfile "SweetYaarDebugger.kicad_sch")
+		(units
+			(unit
+				(name "A")
+				(pins "1" "2")
+			)
+		)
 		(zone_connect 1)
 		(attr exclude_from_bom allow_soldermask_bridges)
@@
 		(sheetname "/")
 		(sheetfile "SweetYaarDebugger.kicad_sch")
+		(units
+			(unit
+				(name "A")
+				(pins "1" "2")
+			)
+		)
 		(zone_connect 1)
 		(attr exclude_from_bom allow_soldermask_bridges)
@@
 			(at 0 -5.645 270)
 			(layer "F.SilkS")
+			(hide yes)
 			(effects
 				(font
@@
 		(sheetname "/")
 		(sheetfile "SweetYaarDebugger.kicad_sch")
+		(units
+			(unit
+				(name "A")
+				(pins "SH" "A1" "A12" "B1" "B12" "A4" "A9" "B4" "B9" "A5" "B5" "A7" "B7"
+					"A6" "B6" "A8" "B8"
+				)
+			)
+		)
 		(attr smd)
 		(duplicate_pad_numbers_are_jumpers no)
@@
 		(sheetname "/")
 		(sheetfile "SweetYaarDebugger.kicad_sch")
+		(units
+			(unit
+				(name "A")
+				(pins "15" "5" "6" "8" "7" "16" "4" "1" "2" "3" "9" "10" "11" "12" "13"
+					"14"
+				)
+			)
+		)
 		(attr smd)
 		(duplicate_pad_numbers_are_jumpers no)
@@
 		(sheetname "/")
 		(sheetfile "SweetYaarDebugger.kicad_sch")
+		(units
+			(unit
+				(name "A")
+				(pins "3" "1" "2")
+			)
+		)
 		(attr smd)
 		(duplicate_pad_numbers_are_jumpers no)
@@
 		(sheetname "/")
 		(sheetfile "SweetYaarDebugger.kicad_sch")
+		(units
+			(unit
+				(name "A")
+				(pins "1" "3" "5" "2" "6" "4")
+			)
+		)
 		(attr smd)
 		(duplicate_pad_numbers_are_jumpers no)
@@
 		(sheetname "/")
 		(sheetfile "SweetYaarDebugger.kicad_sch")
+		(units
+			(unit
+				(name "A")
+				(pins "1" "2")
+			)
+		)
 		(attr smd)
 		(duplicate_pad_numbers_are_jumpers no)
@@
 		(sheetname "/")
 		(sheetfile "SweetYaarDebugger.kicad_sch")
+		(units
+			(unit
+				(name "A")
+				(pins "1" "2")
+			)
+		)
 		(attr smd)
 		(duplicate_pad_numbers_are_jumpers no)
@@
 		(sheetname "/")
 		(sheetfile "SweetYaarDebugger.kicad_sch")
+		(units
+			(unit
+				(name "A")
+				(pins "1" "2")
+			)
+		)
 		(attr smd)
 		(duplicate_pad_numbers_are_jumpers no)
@@
 		(sheetname "/")
 		(sheetfile "SweetYaarDebugger.kicad_sch")
+		(units
+			(unit
+				(name "A")
+				(pins "1" "2")
+			)
+		)
 		(attr smd)
 		(duplicate_pad_numbers_are_jumpers no)
@@
 		(sheetname "/")
 		(sheetfile "SweetYaarDebugger.kicad_sch")
+		(units
+			(unit
+				(name "A")
+				(pins "1" "2")
+			)
+		)
 		(attr smd)
 		(duplicate_pad_numbers_are_jumpers no)
@@
 		(sheetname "/")
 		(sheetfile "SweetYaarDebugger.kicad_sch")
+		(units
+			(unit
+				(name "A")
+				(pins "1" "2")
+			)
+		)
 		(attr smd)
 		(duplicate_pad_numbers_are_jumpers no)
@@
 		(sheetname "/")
 		(sheetfile "SweetYaarDebugger.kicad_sch")
+		(units
+			(unit
+				(name "A")
+				(pins "1" "2")
+			)
+		)
 		(attr smd)
 		(duplicate_pad_numbers_are_jumpers no)
@@
 		(sheetname "/")
 		(sheetfile "SweetYaarDebugger.kicad_sch")
+		(units
+			(unit
+				(name "A")
+				(pins "1" "3" "2")
+			)
+		)
 		(attr smd)
 		(duplicate_pad_numbers_are_jumpers no)
@@
 		(sheetname "/")
 		(sheetfile "SweetYaarDebugger.kicad_sch")
+		(units
+			(unit
+				(name "A")
+				(pins "1" "2")
+			)
+		)
 		(attr smd)
 		(duplicate_pad_numbers_are_jumpers no)
@@
 			)
 		)
-		(property "Value" "2.2uF"
+		(property "Value" "4.7uF"
 			(at 0 1.68 90)
 			(layer "F.SilkS")
@@
 			)
 		)
-		(property "Datasheet" "https://www.lcsc.com/datasheet/C126591.pdf"
+		(property "Datasheet" "https://www.lcsc.com/datasheet/C1779.pdf"
 			(at 0 0 90)
 			(layer "F.Fab")
@@
 			)
 		)
-		(property "LCSC" "C126591"
+		(property "LCSC" "C1779"
 			(at 0 0 270)
 			(unlocked yes)
@@
 		(sheetname "/")
 		(sheetfile "SweetYaarDebugger.kicad_sch")
+		(units
+			(unit
+				(name "A")
+				(pins "1" "2")
+			)
+		)
 		(attr smd)
 		(duplicate_pad_numbers_are_jumpers no)
@@
 			)
 		)
-		(property "Value" "2.2uF"
+		(property "Value" "4.7uF"
 			(at 0 1.68 90)
 			(layer "F.SilkS")
@@
 			)
 		)
-		(property "Datasheet" "https://www.lcsc.com/datasheet/C126591.pdf"
+		(property "Datasheet" "https://www.lcsc.com/datasheet/C1779.pdf"
 			(at 0 0 90)
 			(layer "F.Fab")
@@
 			)
 		)
-		(property "LCSC" "C126591"
+		(property "LCSC" "C1779"
 			(at 0 0 90)
 			(unlocked yes)
@@
 		(sheetname "/")
 		(sheetfile "SweetYaarDebugger.kicad_sch")
+		(units
+			(unit
+				(name "A")
+				(pins "1" "2")
+			)
+		)
 		(attr smd)
 		(duplicate_pad_numbers_are_jumpers no)
@@
 	)
 	(gr_circle
-		(center 113.27 37.08)
-		(end 113.27 37.48)
+		(center 113.23 37.57)
+		(end 113.23 37.97)
 		(stroke
 			(width 0.1)
