File: hardware/mainboard/sweetyaar-mainboard.kicad_pcb (KiCad board)
At the start: 4 copper layers, 80 x 80 mm, 119 parts, among them Q1 MMBT3904

Commit message: removing diode on AUX power; silkscreen changes
Parts:
- removed D2: ESD441, SweetYaar:Texas_DPY0002A_0.6x1mm_P0.65mm
Routing:
- net GND: track 161.8 -> 160.1 mm, vias 71 -> 73
Other:
- board text added: "+"
- board text added: "-"
- board text added: "DIN"
- board text added: "TH"
- board text added: "THERMISTOR BYPASS Disables battery temperature protection. Leave open."
- board text removed: "Close the jumper if no thermistor is connected to the battery harness. This connects a 10k resistor instead which the charger reads as a normal temperature."

Commit message: Creating production v1.0 manufacturing files
Parts:
- C_3V3_OUT1, C_5V_OUT1, C_5V_OUT2: value 22uF, 16 V, X5R/X7R, ±20% -> 22uF, 25 V, X5R, ±10%
- C_BAT_SW_IN1, C_ESP_EN1, C_MUX1, C_MUX2, C_MUX4, C_SD_SW_IN1: value 1uF, 25 V, X7R, ±10% -> 1uF, 50 V, X5R, ±10%
- C_CHG_BAT1, C_MUX3: value 2.2 uF, 25 V, X7R, ±10% -> 4.7 uF, 25 V, X5R, ±10%
